File: io-dev-board.kicad_pcb (KiCad board)
At the start: 2 copper layers, 95.5 x 57.5 mm, 67 parts, among them IC1 24LC01B_P, J1 PWR, J2 SW_Conn, J3 LED_Conn, J4 I2C_Conn, J5 Rot_Conn, Q1 Q_NPN, Q2 Q_NPN, Q3 Q_NPN, Q4 Q_NPN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

Commit message: add '3.3V!' label to board, remove floating 'not connected' mark
Other:
- board text added: "3.3V!"
Changed lines of the file:
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@@
 		(layer "Edge.Cuts")
 	)
+	(gr_text "3.3V!"
+		(at 163 90.5 0)
+		(layer "F.Cu" knockout)
+		(effects
+			(font
+				(size 1.8 1.8)
+				(thickness 0.45)
+				(bold yes)
+			)
+			(justify left bottom)
+		)
+	)
+	(gr_text "3.3V!"
+		(at 163 90.5 0)
+		(layer "F.Mask" knockout)
+		(effects
+			(font
+				(size 1.8 1.8)
+				(thickness 0.45)
+				(bold yes)
+			)
+			(justify left bottom)
+		)
+	)
 	(gr_text "On"
 		(at 169.916985 112.972487 90)
@@
 		(layer "F.Cu")
 		(hatch none 0.1)
-		(priority 30029)
+		(priority 30030)
 		(attr
 			(teardrop
@@
 		(layer "F.Cu")
 		(hatch none 0.1)
-		(priority 30021)
+		(priority 30023)
 		(attr
 			(teardrop
@@
 		(layer "F.Cu")
 		(hatch none 0.1)
-		(priority 30030)
+		(priority 30026)
 		(attr
 			(teardrop
@@
 		(layer "F.Cu")
 		(hatch none 0.1)
-		(priority 30022)
+		(priority 30021)
 		(attr
 			(teardrop
@@
 		(layer "F.Cu")
 		(hatch none 0.1)
-		(priority 30033)
+		(priority 30034)
 		(attr
 			(teardrop
@@
 		(layer "F.Cu")
 		(hatch none 0.1)
-		(priority 30023)
+		(priority 30022)
 		(attr
 			(teardrop
@@
 		(layer "F.Cu")
 		(hatch none 0.1)
-		(priority 30028)
+		(priority 30027)
 		(attr
 			(teardrop
@@
 		(layer "F.Cu")
 		(hatch none 0.1)
-		(priority 30026)
+		(priority 30028)
 		(attr
 			(teardrop
@@
 		(layer "F.Cu")
 		(hatch none 0.1)
-		(priority 30027)
+		(priority 30029)
 		(attr
 			(teardrop
@@
 		(layer "F.Cu")
 		(hatch none 0.1)
-		(priority 30034)
+		(priority 30033)
 		(attr
 			(teardrop

Commit message: fix: pin order for NPN transistors
Parts:
- moved Q1 5.00 mm to (95.0, 111.3), turned to 180 degrees
- moved Q2 5.00 mm to (108.5, 111.3), turned to 180 degrees
- moved Q3 5.00 mm to (122.0, 111.3), turned to 180 degrees
- moved Q4 5.00 mm to (135.5, 111.3), turned to 180 degrees
- moved Q5 5.00 mm to (149.0, 111.3), turned to 180 degrees
Connections:
- Q1 pad 1: Net-(Q1-C) -> GND
- Q1 pad 3: GND -> Net-(Q1-C)
- Q2 pad 1: Net-(Q2-C) -> GND
- Q2 pad 3: GND -> Net-(Q2-E)
- Q3 pad 1: Net-(Q3-C) -> GND
- Q3 pad 3: GND -> Net-(Q3-E)
- Q4 pad 1: Net-(Q4-C) -> GND
- Q4 pad 3: GND -> Net-(Q4-E)
- Q5 pad 1: Net-(Q5-C) -> GND
- Q5 pad 3: GND -> Net-(Q5-E)
- R2 pad 2: Net-(Q2-C) -> Net-(Q2-E)
- R3 pad 2: Net-(Q3-C) -> Net-(Q3-E)
- R4 pad 2: Net-(Q4-C) -> Net-(Q4-E)
- R5 pad 2: Net-(Q5-C) -> Net-(Q5-E)
Routing:
- net Net-(Q4-C): track 8.21 -> 0.00 mm
- net Net-(Q3-C): track 8.21 -> 0.00 mm
- net Net-(Q2-C): track 8.21 -> 0.00 mm
- net Net-(Q5-C): track 8.16 -> 0.00 mm
- net Net-(Q3-E): track 0.00 -> 8.08 mm
- net Net-(Q2-E): track 0.00 -> 8.08 mm
- net Net-(Q5-E): track 0.00 -> 8.08 mm
- net Net-(Q4-E): track 0.00 -> 8.08 mm
